Commit message: Update for collision monitoring

File: catkin_workspace/src/narko_kinova_base_collision/environment/models/narkin/narkin (dual_arm actuator).urdf (robot description, URDF)
Before this commit: robot Narkin, 10 links, 9 joints
Links:
- added link bracelet_link_2nd, mass 0.364; collision mesh filename=package://kortex_description/arms/gen3/7dof/meshes/bracelet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; visual mesh filename=package://kortex_description/arms/gen3/7dof/meshes/bracelet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
- added link forearm_link_2nd, mass 0.9302; collision mesh filename=package://kortex_description/arms/gen3/7dof/meshes/forearm_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; visual mesh filename=package://kortex_description/arms/gen3/7dof/meshes/forearm_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
- added link half_arm_1_link_2nd, mass 1.1636; collision mesh filename=package://kortex_description/arms/gen3/7dof/meshes/half_arm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; visual mesh filename=package://kortex_description/arms/gen3/7dof/meshes/half_arm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
- added link half_arm_2_link_2nd, mass 1.1636; collision mesh filename=package://kortex_description/arms/gen3/7dof/meshes/half_arm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; visual mesh filename=package://kortex_description/arms/gen3/7dof/meshes/half_arm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
- added link kinova_base_link_2, mass 1.697; collision mesh filename=package://kortex_description/arms/gen3/7dof/meshes/base_lin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; visual mesh filename=package://kortex_description/arms/gen3/7dof/meshes/base_lin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
- added link shoulder_link_2nd, mass 1.3773; collision mesh filename=package://kortex_description/arms/gen3/7dof/meshes/shoulder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; visual mesh filename=package://kortex_description/arms/gen3/7dof/meshes/shoulder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
- added link spherical_wrist_1_link_2nd, mass 0.6781; collision mesh filename=package://kortex_description/arms/gen3/7dof/meshes/spherica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; visual mesh filename=package://kortex_description/arms/gen3/7dof/meshes/spherica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
- added link spherical_wrist_2_link_2nd, mass 0.6781; collision mesh filename=package://kortex_description/arms/gen3/7dof/meshes/spherica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; visual mesh filename=package://kortex_description/arms/gen3/7dof/meshes/spherica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
Joints:
- removed joint joint_1
- removed joint joint_2
- removed joint joint_3
- removed joint joint_4
- removed joint joint_5
- removed joint joint_6
- removed joint joint_7
- added joint Actuator1: type continuous, parent kinova_base_link_2, child shoulder_link_2nd, origin xyz=0 0 0.15643 rpy=3.1416 2.7629E-18 -4.9305E-36, axis 0 0 1, limit effort=39 velocity=1.3963
- added joint Actuator2: type revolute, parent shoulder_link_2nd, child half_arm_1_link_2nd, origin xyz=0 0.005375 -0.12838 rpy=1.5708 2.1343E-17 -1.1102E-16, axis 0 0 1, limit lower=-2.41 upper=2.41 effort=39 velocity=1.3963
- added joint Actuator3: type continuous, parent half_arm_1_link_2nd, child half_arm_2_link_2nd, origin xyz=0 -0.21038 -0.006375 rpy=-1.5708 1.2326E-32 -2.9122E-16, axis 0 0 1, limit effort=39 velocity=1.3963
- added joint Actuator4: type revolute, parent half_arm_2_link_2nd, child forearm_link_2nd, origin xyz=0 0.006375 -0.21038 rpy=1.5708 -6.6954E-17 -1.6653E-16, axis 0 0 1, limit lower=-2.66 upper=2.66 effort=39 velocity=1.3963
- added joint Actuator5: type continuous, parent forearm_link_2nd, child spherical_wrist_1_link_2nd, origin xyz=0 -0.20843 -0.006375 rpy=-1.5708 2.2204E-16 -6.373E-17, axis 0 0 1, limit effort=9 velocity=1.2218
- added joint Actuator6: type revolute, parent spherical_wrist_1_link_2nd, child spherical_wrist_2_link_2nd, origin xyz=0 0.00017505 -0.10593 rpy=1.5708 9.2076E-28 -8.2157E-15, axis 0 0 1, limit lower=-2.23 upper=2.23 effort=9 velocity=1.2218
- added joint Actuator7: type continuous, parent spherical_wrist_2_link_2nd, child bracelet_link_2nd, origin xyz=0 -0.10593 -0.00017505 rpy=-1.5708 -5.5511E-17 9.6396E-17, axis 0 0 1, limit effort=9 velocity=1.2218
- added joint joint_9: type fixed, parent narko_base_link, child kinova_base_link_2, origin xyz=0.16 -0.1 0.64 rpy=0 0 0
- joint joint_8: origin xyz=0.16 0.04 0.64 rpy=0 0 0 -> xyz=0.16 0.1 0.64 rpy=0 0 0

File: catkin_workspace/src/narko_kinova_base_collision/environment/models/narkin/narkin.urdf (robot description, URDF)
Before this commit: robot Narkin, 18 links, 17 joints
Links:
- removed link bracelet_link_2nd
- removed link forearm_link_2nd
- removed link half_arm_1_link_2nd
- removed link half_arm_2_link_2nd
- removed link kinova_base_link_2
- removed link shoulder_link_2nd
- removed link spherical_wrist_1_link_2nd
- removed link spherical_wrist_2_link_2nd
- added link link_left_wheel, mass 0.2; collision cylinder length=0.04 radius=0.1
- added link link_right_wheel, mass 0.2; collision cylinder length=0.04 radius=0.1
Joints:
- removed joint joint_1
- removed joint joint_1_2nd
- removed joint joint_2
- removed joint joint_2_2nd
- removed joint joint_3
- removed joint joint_3_2nd
- removed joint joint_4
- removed joint joint_4_2nd
- removed joint joint_5
- removed joint joint_5_2nd
- removed joint joint_6
- removed joint joint_6_2nd
- removed joint joint_7
- removed joint joint_7_2nd
- removed joint joint_9
- added joint Actuator1: type continuous, parent base_link, child shoulder_link, origin xyz=0 0 0.15643 rpy=3.1416 2.7629E-18 -4.9305E-36, axis 0 0 1, limit effort=39 velocity=1.3963
- added joint Actuator2: type revolute, parent shoulder_link, child half_arm_1_link, origin xyz=0 0.005375 -0.12838 rpy=1.5708 2.1343E-17 -1.1102E-16, axis 0 0 1, limit lower=-2.41 upper=2.41 effort=39 velocity=1.3963
- added joint Actuator3: type continuous, parent half_arm_1_link, child half_arm_2_link, origin xyz=0 -0.21038 -0.006375 rpy=-1.5708 1.2326E-32 -2.9122E-16, axis 0 0 1, limit effort=39 velocity=1.3963
- added joint Actuator4: type revolute, parent half_arm_2_link, child forearm_link, origin xyz=0 0.006375 -0.21038 rpy=1.5708 -6.6954E-17 -1.6653E-16, axis 0 0 1, limit lower=-2.66 upper=2.66 effort=39 velocity=1.3963
- added joint Actuator5: type continuous, parent forearm_link, child spherical_wrist_1_link, origin xyz=0 -0.20843 -0.006375 rpy=-1.5708 2.2204E-16 -6.373E-17, axis 0 0 1, limit effort=9 velocity=1.2218
- added joint Actuator6: type revolute, parent spherical_wrist_1_link, child spherical_wrist_2_link, origin xyz=0 0.00017505 -0.10593 rpy=1.5708 9.2076E-28 -8.2157E-15, axis 0 0 1, limit lower=-2.23 upper=2.23 effort=9 velocity=1.2218
- added joint Actuator7: type continuous, parent spherical_wrist_2_link, child bracelet_link, origin xyz=0 -0.10593 -0.00017505 rpy=-1.5708 -5.5511E-17 9.6396E-17, axis 0 0 1, limit effort=9 velocity=1.2218
- added joint joint_left_wheel: type continuous, parent narko_base_link, child link_left_wheel, origin xyz=-0.05 -0.15 0 rpy=0 0 0, axis 0 1 0, limit effort=10000 velocity=1000
- added joint joint_right_wheel: type continuous, parent narko_base_link, child link_right_wheel, origin xyz=-0.05 0.15 0 rpy=0 0 0, axis 0 1 0, limit effort=10000 velocity=1000
- joint joint_8: origin xyz=0.16 0.1 0.64 rpy=0 0 0 -> xyz=-0.15 0.0 0.14 rpy=0 0 0
